File: led-er-v2/led-er-v2.3b.brd (EAGLE design)
At the start: 106.7 x 83.5 mm, 39 parts, among them IC1 TLC59711, IC2 TLC59711, IC3 TLC59711, IC4 TLC59711

Commit message: updated led-er 2.3b
Parts:
- added JP_15VIN1: (no value), microbuilder:1X02_OVAL
- moved JP_SIGOUT 3.19 mm to (104.5, 38.7)
- moved JP_15VIN 2.25 mm to (86.6, 81.3)
- moved C9 0.32 mm to (89.9, 45.7)
- moved JP_SIGIN 0.32 mm to (31.1, 81.4)
- moved JP_5V 0.32 mm to (56.3, 81.3)
Connections:
- net +15V: now also JP_15VIN1.2
- net GND: now also JP_15VIN1.1
Routing:
- net +15V: track 78.1 -> 85.1 mm
- net VCC: track 19.7 -> 23.6 mm
- net N$60: track 19.4 -> 22.6 mm
- net N$59: track 15.3 -> 18.5 mm
- net N$61: track 28.9 -> 30.5 mm
- net N$57: track 8.34 -> 6.85 mm
- net N$62: track 29.2 -> 30.5 mm
- net N$58: track 8.29 -> 7.00 mm
- net N$56: track 8.31 -> 7.35 mm
- net N$4: track 29.1 -> 30.0 mm
- net SCKI: track 88.4 -> 87.5 mm
- net SDTI: track 105.2 -> 106.0 mm
- net N$71: track 26.0 -> 26.7 mm
- net SCKO3: track 20.7 -> 20.0 mm
- net SCKO1: track 23.4 -> 22.8 mm
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