File: led-er-v3/led-er-v3-module-d.sch (EAGLE design)
At the start: 17 parts

Commit message: long and skinny working
Parts:
- added JP1, JP2, JP3: (no value), Andrews:HEADER_SMD_2_MALESMD-STRAIGHT-ALT-FEMALE
Connections:
- new net N$2: JP1.2
- new net N$3: JP1.1
- new net N$4: JP2.2
- new net N$5: JP2.1
- new net N$6: JP3.2
- new net N$7: JP3.1
