File: led-er-v3/led-er-v3-module-e.sch (EAGLE design)
At the start: 20 parts

Commit message: long and skinny working
Parts:
- removed JP1, JP2, JP3: (no value), Andrews:HEADER_SMD_2_MALESMD-STRAIGHT-FEMALE
Connections:
- removed net N$2: JP1.2
- removed net N$3: JP1.1
- removed net N$4: JP2.2
- removed net N$5: JP2.1
- removed net N$6: JP3.2
- removed net N$7: JP3.1
Changed lines of the file:
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@@
 <?xml version="1.0" encoding="utf-8"?>
 <!DOCTYPE eagle SYSTEM "eagle.dtd">
-<eagle version="7.5.0">
+<eagle version="7.2.0">
 <drawing>
 <settings>
@@
 <layer number="56" name="wert" color="7" fill="1" visible="no" active="no"/>
 <layer number="57" name="tCAD" color="7" fill="1" visible="no" active="no"/>
-<layer number="59" name="tCarbon" color="7" fill="1" visible="no" active="no"/>
-<layer number="60" name="bCarbon" color="7" fill="1" visible="no" active="no"/>
 <layer number="90" name="Modules" color="5" fill="1" visible="yes" active="yes"/>
 <layer number="91" name="Nets" color="2" fill="1" visible="yes" active="yes"/>
@@
 <layer number="112" name="tSilk" color="7" fill="1" visible="yes" active="yes"/>
 <layer number="113" name="ReferenceLS" color="7" fill="1" visible="no" active="no"/>
-<layer number="114" name="Badge_Outline" color="7" fill="1" visible="yes" active="yes"/>
-<layer number="115" name="ReferenceISLANDS" color="7" fill="1" visible="yes" active="yes"/>
 <layer number="116" name="Patch_BOT" color="9" fill="4" visible="yes" active="yes"/>
 <layer number="118" name="Rect_Pads" color="7" fill="1" visible="no" active="no"/>
@@
 <layer number="127" name="_tValues" color="7" fill="1" visible="yes" active="yes"/>
 <layer number="128" name="_bValues" color="7" fill="1" visible="yes" active="yes"/>
-<layer number="129" name="Mask" color="7" fill="1" visible="yes" active="yes"/>
 <layer number="131" name="tAdjust" color="7" fill="1" visible="no" active="yes"/>
 <layer number="132" name="bAdjust" color="7" fill="1" visible="no" active="yes"/>
@@
 <layer number="223" name="223bmp" color="24" fill="1" visible="no" active="no"/>
 <layer number="224" name="224bmp" color="25" fill="1" visible="no" active="no"/>
-<layer number="225" name="225bmp" color="7" fill="1" visible="yes" active="yes"/>
-<layer number="226" name="226bmp" color="7" fill="1" visible="yes" active="yes"/>
-<layer number="227" name="227bmp" color="7" fill="1" visible="yes" active="yes"/>
-<layer number="228" name="228bmp" color="7" fill="1" visible="yes" active="yes"/>
-<layer number="229" name="229bmp" color="7" fill="1" visible="yes" active="yes"/>
-<layer number="230" name="230bmp" color="7" fill="1" visible="yes" active="yes"/>
 <layer number="231" name="Eagle3D_PG1" color="7" fill="1" visible="no" active="no"/>
 <layer number="232" name="Eagle3D_PG2" color="7" fill="1" visible="no" active="no"/>
@@
 <layer number="251" name="SMDround" color="7" fill="1" visible="no" active="no"/>
 <layer number="254" name="cooling" color="7" fill="1" visible="yes" active="yes"/>
-<layer number="255" name="routoute" color="7" fill="1" visible="yes" active="yes"/>
 </layers>
 <schematic xreflabel="%F%N/%S.%C%R" xrefpart="/%S.%C%R">
@@
 <part name="U$2" library="microbuilder" deviceset="MOUNTINGHOLE" device=""/>
 <part name="U$4" library="microbuilder" deviceset="MOUNTINGHOLE" device=""/>
-<part name="JP1" library="Andrews" deviceset="HEADER_SMD_2_MALE" device="SMD-STRAIGHT-FEMALE"/>
-<part name="JP2" library="Andrews" deviceset="HEADER_SMD_2_MALE" device="SMD-STRAIGHT-FEMALE"/>
-<part name="JP3" library="Andrews" deviceset="HEADER_SMD_2_MALE" device="SMD-STRAIGHT-FEMALE"/>
 </parts>
 <sheets>
@@
 <instance part="U$2" gate="G$1" x="-30.48" y="-40.64" rot="R90"/>
 <instance part="U$4" gate="G$1" x="-30.48" y="-55.88" rot="R90"/>
-<instance part="JP1" gate="G$1" x="121.92" y="-20.32" rot="R90"/>
-<instance part="JP2" gate="G$1" x="167.64" y="-20.32" rot="R90"/>
-<instance part="JP3" gate="G$1" x="213.36" y="-20.32" rot="R90"/>
 </instances>
 <busses>
@@
 <portref moduleinst="LED-ER1" port="2SCKO"/>
 <portref moduleinst="LED-ER2" port="1SCKI"/>
-<wire x1="119.38" y1="2.54" x2="121.92" y2="2.54" width="0.1524" layer="91"/>
-<pinref part="JP1" gate="G$1" pin="2"/>
-<wire x1="121.92" y1="2.54" x2="124.46" y2="2.54" width="0.1524" layer="91"/>
-<wire x1="121.92" y1="-15.24" x2="121.92" y2="2.54" width="0.1524" layer="91"/>
-<junction x="121.92" y="2.54"/>
+<wire x1="119.38" y1="2.54" x2="124.46" y2="2.54" width="0.1524" layer="91"/>
 </segment>
 </net>
@@
 <portref moduleinst="LED-ER2" port="1SDTI"/>
 <wire x1="119.38" y1="-2.54" x2="124.46" y2="-2.54" width="0.1524" layer="91"/>
-<pinref part="JP1" gate="G$1" pin="1"/>
-<wire x1="124.46" y1="-15.24" x2="124.46" y2="-2.54" width="0.1524" layer="91"/>
-<junction x="124.46" y="-2.54"/>
 </segment>
 </net>
@@
 <portref moduleinst="LED-ER2" port="2SCKO"/>
 <portref moduleinst="LED-ER3" port="1SCKI"/>
-<wire x1="165.1" y1="2.54" x2="167.64" y2="2.54" width="0.1524" layer="91"/>
-<pinref part="JP2" gate="G$1" pin="2"/>
-<wire x1="167.64" y1="2.54" x2="170.18" y2="2.54" width="0.1524" layer="91"/>
-<wire x1="167.64" y1="-15.24" x2="167.64" y2="2.54" width="0.1524" layer="91"/>
-<junction x="167.64" y="2.54"/>
+<wire x1="165.1" y1="2.54" x2="170.18" y2="2.54" width="0.1524" layer="91"/>
 </segment>
 </net>
@@
 <portref moduleinst="LED-ER3" port="1SDTI"/>
 <wire x1="165.1" y1="-2.54" x2="170.18" y2="-2.54" width="0.1524" layer="91"/>
-<pinref part="JP2" gate="G$1" pin="1"/>
-<wire x1="170.18" y1="-15.24" x2="170.18" y2="-2.54" width="0.1524" layer="91"/>
-<junction x="170.18" y="-2.54"/>
 </segment>
 </net>
@@
 <portref moduleinst="LED-ER3" port="2SCKO"/>
 <portref moduleinst="LED-ER4" port="1SCKI"/>
-<wire x1="210.82" y1="2.54" x2="213.36" y2="2.54" width="0.1524" layer="91"/>
-<pinref part="JP3" gate="G$1" pin="2"/>
-<wire x1="213.36" y1="2.54" x2="215.9" y2="2.54" width="0.1524" layer="91"/>
-<wire x1="213.36" y1="-15.24" x2="213.36" y2="2.54" width="0.1524" layer="91"/>
-<junction x="213.36" y="2.54"/>
+<wire x1="210.82" y1="2.54" x2="215.9" y2="2.54" width="0.1524" layer="91"/>
 </segment>
 </net>
@@
 <portref moduleinst="LED-ER4" port="1SDTI"/>
 <wire x1="210.82" y1="-2.54" x2="215.9" y2="-2.54" width="0.1524" layer="91"/>
-<pinref part="JP3" gate="G$1" pin="1"/>
-<wire x1="215.9" y1="-15.24" x2="215.9" y2="-2.54" width="0.1524" layer="91"/>
-<junction x="215.9" y="-2.54"/>
-</segment>
-</net>
+</segment>
+</net>
