File: led-er-v3/led-er-v3-module-f.brd (EAGLE design)
At the start: 159.3 x 53.2 mm, 44 parts

Commit message: updated
Parts:
- removed JP_SIGIN: (no value), microbuilder:1X02_OVAL
- added JP_SIG_IN: (no value), Andrews:1X06_SMD_STRAIGHT_ALT
Connections:
- net 1SCKI: now also JP_SIG_IN.2; no longer JP_SIGIN.2
- net 1SDTI: now also JP_SIG_IN.1; no longer JP_SIGIN.1
Routing:
- net 1SDTI: track 84.8 -> 23.3 mm
- net 1SCKI: track 50.1 -> 43.6 mm
Changed lines of the file:
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@@
 <attribute name="VALUE" x="15.793721875" y="54.4139125" size="0.4064" layer="27" ratio="10" rot="R180"/>
-</element>
-<element name="JP_SIGIN" library="microbuilder" package="1X02_OVAL" value="" x="127.701140625" y="46.40370625" smashed="yes" rot="R180">
-<attribute name="VALUE" x="130.241140625" y="49.57870625" size="0.4064" layer="27" ratio="10" rot="R180"/>
 </element>
 <element name="LED-ER1:TLC1" library="adafruit" package="HTSSOP20DAP" value="TLC59711" x="99.058475" y="43.95520625" rot="R90"/>
@@
 <attribute name="PROD_ID" value="CONN-10203" x="36.316246875" y="46.56230625" size="1.778" layer="27" display="off"/>
 <attribute name="VALUE" x="32.506246875" y="42.37130625" size="1.27" layer="27"/>
+</element>
+<element name="JP_SIG_IN" library="Andrews" package="1X06_SMD_STRAIGHT_ALT" value="" x="113.26158125" y="46.560553125">
+<attribute name="PROD_ID" value="CONN-10203" x="113.26158125" y="46.560553125" size="1.778" layer="27" display="off"/>
 </element>
 </elements>
@@
 <signal name="1SDTI">
 <contactref element="U$5" pad="11"/>
-<contactref element="JP_SIGIN" pad="1"/>
 <contactref element="LED-ER1:TLC1" pad="9"/>
-<wire x1="101.858475" y1="46.23020625" x2="114.620371875" y2="46.23020625" width="0.3048" layer="1"/>
+<wire x1="101.858475" y1="46.23020625" x2="113.26158125" y2="46.23020625" width="0.3048" layer="1"/>
+<wire x1="113.26158125" y1="46.23020625" x2="114.620371875" y2="46.23020625" width="0.3048" layer="1"/>
 <wire x1="116.367971875" y1="44.38335625" x2="116.845746875" y2="43.90558125" width="0.6096" layer="1"/>
 <wire x1="116.845746875" y1="43.90558125" x2="119.306728125" y2="41.4446" width="0.6096" layer="1"/>
 <wire x1="119.306728125" y1="41.4446" x2="119.306728125" y2="39.582221875" width="0.6096" layer="1"/>
 <wire x1="119.306728125" y1="39.582221875" x2="119.2982125" y2="39.57370625" width="0.3048" layer="1"/>
-<wire x1="128.971140625" y1="46.40370625" x2="128.971140625" y2="43.927371875" width="0.6096" layer="1"/>
-<wire x1="128.971140625" y1="43.927371875" x2="122.947175" y2="38.22191875" width="0.6096" layer="1"/>
-<wire x1="122.947175" y1="38.22191875" x2="122.947175" y2="26.436828125" width="0.6096" layer="1"/>
-<wire x1="122.947175" y1="26.436828125" x2="117.85091875" y2="21.340571875" width="0.6096" layer="1"/>
-<wire x1="117.85091875" y1="21.340571875" x2="115.62130625" y2="21.340571875" width="0.6096" layer="1"/>
-<wire x1="115.62130625" y1="21.340571875" x2="114.665759375" y2="22.29611875" width="0.6096" layer="1"/>
-<wire x1="114.665759375" y1="22.29611875" x2="114.665759375" y2="26.118309375" width="0.6096" layer="1"/>
-<wire x1="114.665759375" y1="26.118309375" x2="115.621309375" y2="27.167496875" width="0.6096" layer="1"/>
-<wire x1="115.621309375" y1="27.167496875" x2="118.48795" y2="27.167496875" width="0.6096" layer="1"/>
-<wire x1="118.48795" y1="27.167496875" x2="119.762015625" y2="28.347925" width="0.6096" layer="1"/>
-<wire x1="119.762015625" y1="28.347925" x2="119.762015625" y2="32.80715" width="0.6096" layer="1"/>
-<wire x1="119.762015625" y1="32.80715" x2="113.7102125" y2="38.858953125" width="0.6096" layer="1"/>
-<wire x1="113.7102125" y1="38.858953125" x2="113.7102125" y2="41.725596875" width="0.6096" layer="1"/>
-<wire x1="113.7102125" y1="41.725596875" x2="116.367971875" y2="44.38335625" width="0.6096" layer="1"/>
 <wire x1="114.620371875" y1="46.23020625" x2="114.984275" y2="45.866303125" width="0.3048" layer="1"/>
 <wire x1="114.984275" y1="45.866303125" x2="116.845746875" y2="43.90558125" width="0.6096" layer="1"/>
+<contactref element="JP_SIG_IN" pad="1"/>
+<wire x1="113.26158125" y1="44.910553125" x2="113.26158125" y2="46.23020625" width="0.3048" layer="1"/>
 </signal>
 <signal name="1SCKI">
 <contactref element="U$5" pad="13"/>
-<contactref element="JP_SIGIN" pad="2"/>
 <contactref element="LED-ER1:TLC1" pad="10"/>
-<wire x1="101.858475" y1="46.88020625" x2="116.518503125" y2="46.88020625" width="0.3048" layer="1"/>
-<wire x1="116.518503125" y1="46.88020625" x2="119.762015625" y2="43.63669375" width="0.6096" layer="1"/>
-<wire x1="119.762015625" y1="43.63669375" x2="121.354596875" y2="42.0441125" width="0.6096" layer="1"/>
+<wire x1="101.858475" y1="46.88020625" x2="110.72158125" y2="46.88020625" width="0.3048" layer="1"/>
+<wire x1="110.72158125" y1="46.88020625" x2="116.518503125" y2="46.88020625" width="0.3048" layer="1"/>
+<wire x1="116.518503125" y1="46.88020625" x2="121.354596875" y2="42.0441125" width="0.6096" layer="1"/>
 <wire x1="121.354596875" y1="42.0441125" x2="121.354596875" y2="27.009065625" width="0.6096" layer="1"/>
 <wire x1="121.354596875" y1="27.009065625" x2="118.676315625" y2="24.330784375" width="0.6096" layer="1"/>
 <wire x1="118.676315625" y1="24.330784375" x2="116.761134375" y2="24.330784375" width="0.6096" layer="1"/>
 <wire x1="116.761134375" y1="24.330784375" x2="116.7582125" y2="24.33370625" width="0.3048" layer="1"/>
-<wire x1="126.431140625" y1="46.40370625" x2="122.529028125" y2="46.40370625" width="0.6096" layer="1"/>
-<wire x1="122.529028125" y1="46.40370625" x2="119.762015625" y2="43.63669375" width="0.6096" layer="1"/>
+<contactref element="JP_SIG_IN" pad="2"/>
+<wire x1="110.72158125" y1="48.210553125" x2="110.72158125" y2="46.88020625" width="0.3048" layer="1"/>
 </signal>
 <signal name="+5V">
@@
 <contactref element="U$5" pad="GND2"/>
 <contactref element="JP_PROG" pad="1"/>
-<wire x1="116.7582125" y1="31.95370625" x2="115.404896875" y2="31.95370625" width="0.4064" layer="1"/>
 <wire x1="115.404896875" y1="31.95370625" x2="112.436146875" y2="28.98495625" width="0.4064" layer="1"/>
 <wire x1="112.436146875" y1="28.98495625" x2="112.436146875" y2="20.385025" width="0.4064" layer="1"/>
@@
 <wire x1="140.46555625" y1="39.8145" x2="140.46555625" y2="46.185978125" width="0.4064" layer="1"/>
 <wire x1="140.46555625" y1="46.185978125" x2="140.51035" y2="46.230771875" width="0.4064" layer="1"/>
+<wire x1="115.404896875" y1="31.95370625" x2="116.7582125" y2="31.95370625" width="0.4064" layer="1"/>
 </signal>
 <signal name="N$55">
